Commit message: docs: add teaching comments across all 4 packages and reorder Stage 2 URDF
Comment every authored source file with file headers and section comments
explaining the ROS 2 concepts behind each block:

- 01_talker_listener: pub/sub role docstrings, queue-depth and entry-point notes
- 02_four_wheeled_robot_urdf: frame conventions, per-wheel mirroring geometry
- 03_four_wheeled_robot_xacro: inertia formulas, include ordering, xacro
  Command()/ParameterValue handoff in the launch file
- 04_four_wheeled_robot_teleop: per-block walkthrough of the differential
  drive kinematics in diff_drive_sim.py, and the mutual exclusion of the
  two /joint_states publishers in the launch file

Rearrange four_wheeled_robot.urdf so all <link> declarations precede all
<joint> declarations, grouping the parts separately from the assembly.
URDF is a graph format, so declaration order is cosmetic; parsed XML
confirms identical links, joints, materials, and parent/child topology.

No executable content changed: verified by comparing Python token streams
(comments and docstrings stripped) and XML element/attribute trees against
the previous revision for all 28 files.

File: src/03_four_wheeled_robot_xacro/urdf/chassis.xacro (robot description, xacro)
@@ -1,5 +1,12 @@
 <?xml version="1.0"?>
+<!--
+  Stage 3: the robot body — base_footprint (ground frame) and base_link
+  (chassis box). All numbers come from properties.xacro, so nothing here
+  needs editing to resize the robot.
+-->
 <robot xmlns:xacro="http://www.ros.org/wiki/xacro">
+  <!-- Dummy frame pinned to the floor; RViz uses it as the fixed frame. -->
   <link name="base_footprint"/>
+  <!-- Fixed joint that lifts the chassis to its riding height. -->
   <joint name="base_footprint_joint" type="fixed">
     <parent link="base_footprint"/>
@@ -8,4 +15,5 @@
   </joint>
   <link name="base_link">
+    <!-- Visual: what RViz draws (same box as the collision volume). -->
     <visual>
       <origin xyz="0 0 0" rpy="0 0 0"/>
@@ -15,4 +23,5 @@
       <material name="blue"/>
     </visual>
+    <!-- Collision: the volume a physics engine / planner would use. -->
     <collision>
       <origin xyz="0 0 0" rpy="0 0 0"/>
@@ -21,4 +30,5 @@
       </geometry>
     </collision>
+    <!-- Inertia is generated from the same dimensions and mass. -->
     <xacro:box_inertia m="${chassis_mass}" x="${chassis_length}" y="${chassis_width}" z="${chassis_height}"/>
   </link>

File: src/03_four_wheeled_robot_xacro/urdf/materials.xacro (robot description, xacro)
@@ -1,3 +1,8 @@
 <?xml version="1.0"?>
+<!--
+  Stage 3: named RGBA colours shared by chassis.xacro and wheel.xacro.
+  Materials are looked up by name from the <visual> tags, so a colour only
+  needs to change in this one file. Alpha is always 1.0 (fully opaque).
+-->
 <robot xmlns:xacro="http://www.ros.org/wiki/xacro">
   <material name="blue">

File: src/03_four_wheeled_robot_xacro/urdf/properties.xacro (robot description, xacro)
@@ -1,5 +1,13 @@
 <?xml version="1.0"?>
+<!--
+  Stage 3: single source of truth for every physical property of the robot.
+  These xacro properties are textual substitutions: the value is pasted into
+  the expression *before* it is evaluated, so ${m/12.0} below computes on
+  numbers, not on strings. Include this file before using any of the names.
+-->
 <robot xmlns:xacro="http://www.ros.org/wiki/xacro">
+  <!-- Pi, needed for the wheel cylinder roll angle (pi/2 = 90 deg). -->
   <xacro:property name="pi_val" value="3.1415926535897931"/>
+  <!-- Chassis box: 0.5 x 0.3 x 0.15 m, 5 kg, raised 0.10 m above the ground. -->
   <xacro:property name="chassis_length" value="0.5"/>
   <xacro:property name="chassis_width" value="0.3"/>
@@ -7,10 +15,16 @@
   <xacro:property name="chassis_mass" value="5.0"/>
   <xacro:property name="chassis_elevation" value="0.10"/>
+  <!-- Wheels: 0.08 m radius, 0.05 m thick, 0.5 kg each. -->
   <xacro:property name="wheel_radius" value="0.08"/>
   <xacro:property name="wheel_width" value="0.05"/>
   <xacro:property name="wheel_mass" value="0.5"/>
+  <!-- Wheel mounting offsets from base_link. Halves of the wheelbase (0.30 m)
+       and track width (0.37 m); -0.02 keeps the wheels just below the box. -->
   <xacro:property name="wheel_offset_x" value="0.15"/>
   <xacro:property name="wheel_offset_y" value="0.185"/>
   <xacro:property name="wheel_offset_z" value="-0.02"/>
+  <!-- Inertia macro for a solid box of mass m and full side lengths x, y, z.
+       Diagonal-only tensor: Ixx=m/12*(y^2+z^2), Iyy=m/12*(x^2+z^2),
+       Izz=m/12*(x^2+y^2); the products of inertia are zero for a box. -->
   <xacro:macro name="box_inertia" params="m x y z">
     <inertial>
@@ -21,4 +35,6 @@
     </inertial>
   </xacro:macro>
+  <!-- Inertia macro for a solid cylinder whose spin axis is local Y.
+       Transverse: Ixx=Izz=m/12*(3r^2+h^2); axial: Iyy=m/2*r^2. -->
   <xacro:macro name="cylinder_inertia" params="m r h">
     <inertial>

File: src/03_four_wheeled_robot_xacro/urdf/robot.urdf.xacro (robot description, xacro)
@@ -1,8 +1,20 @@
 <?xml version="1.0"?>
+<!--
+  Stage 3 top-level robot file: include the parts, then instantiate them.
+  Run `xacro robot.urdf.xacro` to see the flattened plain URDF this produces.
+  Include order matters: properties.xacro must define the dimensions and the
+  inertia macros before chassis.xacro / wheel.xacro use them.
+-->
 <robot xmlns:xacro="http://www.ros.org/wiki/xacro" name="four_wheeled_robot">
+  <!-- Dimensions, masses, and inertia macros. -->
   <xacro:include filename="properties.xacro"/>
+  <!-- Named colours. -->
   <xacro:include filename="materials.xacro"/>
+  <!-- base_footprint + base_link chassis. -->
   <xacro:include filename="chassis.xacro"/>
+  <!-- The reusable wheel macro. -->
   <xacro:include filename="wheel.xacro"/>
+  <!-- Four macro calls: front/rear come from the sign of x_offset, left/right
+       from the sign of y_offset. Y is negated for the right-hand side. -->
   <xacro:wheel name="front_left_wheel" parent="base_link" x_offset="${wheel_offset_x}" y_offset="${wheel_offset_y}" z_offset="${wheel_offset_z}"/>
   <xacro:wheel name="front_right_wheel" parent="base_link" x_offset="${wheel_offset_x}" y_offset="-${wheel_offset_y}" z_offset="${wheel_offset_z}"/>

File: src/03_four_wheeled_robot_xacro/urdf/wheel.xacro (robot description, xacro)
@@ -1,4 +1,13 @@
 <?xml version="1.0"?>
+<!--
+  Stage 3: reusable `wheel` macro.
+  Calling <xacro:wheel name="..." parent="..." x_offset=... y_offset=...
+  z_offset=.../> expands to one continuous joint plus one cylinder link, so
+  all four wheels stay geometrically identical by construction.
+-->
 <robot xmlns:xacro="http://www.ros.org/wiki/xacro">
+  <!-- name: prefix for the joint/link names (e.g. front_left_wheel).
+       parent: chassis link the wheel hangs off.
+       *_offset: mounting position of the wheel centre in the parent frame. -->
   <xacro:macro name="wheel" params="name parent x_offset y_offset z_offset">
     <joint name="${name}_joint" type="continuous">
@@ -6,8 +15,12 @@
       <parent link="${parent}"/>
       <child link="${name}_link"/>
+      <!-- Rotate about local Y: the wheel axle points sideways. -->
       <axis xyz="0 1 0"/>
+      <!-- No position limits (continuous); only effort/velocity caps. -->
       <limit effort="10.0" velocity="20.0"/>
     </joint>
     <link name="${name}_link">
+      <!-- URDF cylinders are built along Z, so roll by 90 deg to align the
+           cylinder axis with the joint's Y rotation axis. -->
       <visual>
         <origin xyz="0 0 0" rpy="${pi_val/2} 0 0"/>

File: src/04_four_wheeled_robot_teleop/urdf/chassis.xacro (robot description, xacro)
@@ -1,5 +1,14 @@
 <?xml version="1.0"?>
+<!--
+  Stage 4: the robot body — base_footprint (ground frame) and base_link
+  (chassis box).
+  base_footprint is the frame diff_drive_sim.py drives with its odom -> ... TF
+  broadcast, so keep this link name stable. Dimensions come from
+  properties.xacro.
+-->
 <robot xmlns:xacro="http://www.ros.org/wiki/xacro">
+  <!-- Dummy frame at floor level; the odom TF lands here. -->
   <link name="base_footprint"/>
+  <!-- Fixed joint that lifts the chassis to its riding height. -->
   <joint name="base_footprint_joint" type="fixed">
     <parent link="base_footprint"/>
@@ -8,4 +17,5 @@
   </joint>
   <link name="base_link">
+    <!-- Visual: what RViz draws (same box as the collision volume). -->
     <visual>
       <origin xyz="0 0 0" rpy="0 0 0"/>
@@ -15,4 +25,5 @@
       <material name="blue"/>
     </visual>
+    <!-- Collision: the volume a physics engine / planner would use. -->
     <collision>
       <origin xyz="0 0 0" rpy="0 0 0"/>
@@ -21,4 +32,5 @@
       </geometry>
     </collision>
+    <!-- Inertia is generated from the same dimensions and mass. -->
     <xacro:box_inertia m="${chassis_mass}" x="${chassis_length}" y="${chassis_width}" z="${chassis_height}"/>
   </link>

File: src/04_four_wheeled_robot_teleop/urdf/materials.xacro (robot description, xacro)
@@ -1,3 +1,8 @@
 <?xml version="1.0"?>
+<!--
+  Stage 4: named RGBA colours shared by chassis.xacro and wheel.xacro.
+  Materials are looked up by name from the <visual> tags, so the chassis
+  colour can be changed here without touching the geometry.
+-->
 <robot xmlns:xacro="http://www.ros.org/wiki/xacro">
   <material name="blue">

File: src/04_four_wheeled_robot_teleop/urdf/properties.xacro (robot description, xacro)
@@ -1,5 +1,14 @@
 <?xml version="1.0"?>
+<!--
+  Stage 4: robot dimensions, masses, and inertia macros.
+  These values are the contract between the model and diff_drive_sim.py:
+  `wheel_radius` (0.08) and the track width 2 * `wheel_offset_y` (0.37) must
+  match that node's parameters, otherwise the simulated motion will not line
+  up with the drawn wheels.
+-->
 <robot xmlns:xacro="http://www.ros.org/wiki/xacro">
+  <!-- Pi, needed for the wheel cylinder roll angle (pi/2 = 90 deg). -->
   <xacro:property name="pi_val" value="3.1415926535897931"/>
+  <!-- Chassis box: 0.5 x 0.3 x 0.15 m, 5 kg, raised 0.10 m above the ground. -->
   <xacro:property name="chassis_length" value="0.5"/>
   <xacro:property name="chassis_width" value="0.3"/>
@@ -7,10 +16,16 @@
   <xacro:property name="chassis_mass" value="5.0"/>
   <xacro:property name="chassis_elevation" value="0.10"/>
+  <!-- Wheels: 0.08 m radius, 0.05 m thick, 0.5 kg each. -->
   <xacro:property name="wheel_radius" value="0.08"/>
   <xacro:property name="wheel_width" value="0.05"/>
   <xacro:property name="wheel_mass" value="0.5"/>
+  <!-- Wheel mounting offsets from base_link. Halves of the wheelbase (0.30 m)
+       and track width (0.37 m); -0.02 keeps the wheels just below the box. -->
   <xacro:property name="wheel_offset_x" value="0.15"/>
   <xacro:property name="wheel_offset_y" value="0.185"/>
   <xacro:property name="wheel_offset_z" value="-0.02"/>
+  <!-- Inertia macro for a solid box of mass m and full side lengths x, y, z.
+       Diagonal-only tensor: Ixx=m/12*(y^2+z^2), Iyy=m/12*(x^2+z^2),
+       Izz=m/12*(x^2+y^2); the products of inertia are zero for a box. -->
   <xacro:macro name="box_inertia" params="m x y z">
     <inertial>
@@ -21,4 +36,6 @@
     </inertial>
   </xacro:macro>
+  <!-- Inertia macro for a solid cylinder whose spin axis is local Y.
+       Transverse: Ixx=Izz=m/12*(3r^2+h^2); axial: Iyy=m/2*r^2. -->
   <xacro:macro name="cylinder_inertia" params="m r h">
     <inertial>

File: src/04_four_wheeled_robot_teleop/urdf/robot.urdf.xacro (robot description, xacro)
@@ -1,8 +1,20 @@
 <?xml version="1.0"?>
+<!--
+  Stage 4 top-level robot file: include the parts, then instantiate them.
+  Identical in structure to Stage 3; the difference in this package is the
+  diff_drive_sim.py node, which animates these same joints and frames.
+  Run `xacro robot.urdf.xacro` to see the flattened plain URDF.
+-->
 <robot xmlns:xacro="http://www.ros.org/wiki/xacro" name="four_wheeled_robot">
+  <!-- Dimensions, masses, and the inertia macros (must come first). -->
   <xacro:include filename="properties.xacro"/>
+  <!-- Named colours. -->
   <xacro:include filename="materials.xacro"/>
+  <!-- base_footprint + base_link chassis. -->
   <xacro:include filename="chassis.xacro"/>
+  <!-- The reusable wheel macro. -->
   <xacro:include filename="wheel.xacro"/>
+  <!-- Four macro calls: front/rear come from the sign of x_offset, left/right
+       from the sign of y_offset. Y is negated for the right-hand side. -->
   <xacro:wheel name="front_left_wheel" parent="base_link" x_offset="${wheel_offset_x}" y_offset="${wheel_offset_y}" z_offset="${wheel_offset_z}"/>
   <xacro:wheel name="front_right_wheel" parent="base_link" x_offset="${wheel_offset_x}" y_offset="-${wheel_offset_y}" z_offset="${wheel_offset_z}"/>

File: src/04_four_wheeled_robot_teleop/urdf/wheel.xacro (robot description, xacro)
@@ -1,4 +1,14 @@
 <?xml version="1.0"?>
+<!--
+  Stage 4: reusable `wheel` macro.
+  One call produces the continuous joint and cylinder link for a single
+  wheel. The resulting joint names (${name}_joint) are exactly what
+  diff_drive_sim.py publishes in its /joint_states message, so renaming a
+  wheel here means updating that node too.
+-->
 <robot xmlns:xacro="http://www.ros.org/wiki/xacro">
+  <!-- name: prefix for the joint/link names (e.g. front_left_wheel).
+       parent: chassis link the wheel hangs off.
+       *_offset: mounting position of the wheel centre in the parent frame. -->
   <xacro:macro name="wheel" params="name parent x_offset y_offset z_offset">
     <joint name="${name}_joint" type="continuous">
@@ -6,8 +16,12 @@
       <parent link="${parent}"/>
       <child link="${name}_link"/>
+      <!-- Rotate about local Y: the wheel axle points sideways. -->
       <axis xyz="0 1 0"/>
+      <!-- No position limits (continuous); only effort/velocity caps. -->
       <limit effort="10.0" velocity="20.0"/>
     </joint>
     <link name="${name}_link">
+      <!-- URDF cylinders are built along Z, so roll by 90 deg to align the
+           cylinder axis with the joint's Y rotation axis. -->
       <visual>
         <origin xyz="0 0 0" rpy="${pi_val/2} 0 0"/>
